File: NeonPine.kicad_sch (KiCad schematic)
At the start: 95 parts, among them J1 USB-C 6P (USB4125-GF-A), J2 SWD pogo pads, Q1 DMN15H310SE, Q11 MMDT5551, Q12 MMDT5551, Q13 MMDT5551, Q14 MMDT5551, Q15 MMDT5551, Q16 MMDT5551, Q17 MMDT5551, Q18 MMDT5551, Q19 MMDT5551, Q2 TEPT4400, Q20 MMDT5551, U1 CH32V003F4P6, U2 74HC595BQ, U3 74HC595BQ

Commit message: finished routing, check and sim
Parts:
- added R13: 33, Resistor_SMD:R_0402_1005Metric, symbol Device:R
Connections:
- net LAMP6: now also U1.3 (PD6); no longer U1.16 (PC6)
- net LAMP9: now also U1.5 (PA1); no longer U1.15 (PC5)
- net SR_CLK: now also R13.2; no longer U1.5 (PA1)
- net SR_DATA: now also U1.16 (PC6); no longer U1.3 (PD6)
- new net SR_SCK: R13.1, U1.15 (PC5)
Other:
- note added: "SR_DATA = PC6 (SPI1 MOSI), SR_CLK = PC5 (SPI1 SCK), SR_LATCH = PD4. /OE tied low: outputs are random until the first latch, but the boost is off then (R2)."
- note removed: "SR_DATA = PD6, SR_CLK = PA1, SR_LATCH = PD4. /OE tied low: outputs are random until the first latch, but the boost is off then (R2)."
Changed lines of the file:
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@@
 		)
 	)
-	(text "SR_DATA = PD6, SR_CLK = PA1, SR_LATCH = PD4. /OE tied low: outputs are random until the first latch, but the boost is off then (R2)."
+	(text "SR_DATA = PC6 (SPI1 MOSI), SR_CLK = PC5 (SPI1 SCK), SR_LATCH = PD4. /OE tied low: outputs are random until the first latch, but the boost is off then (R2)."
 		(exclude_from_sim no)
 		(at 228.6 100.33 0)
@@
 	(wire
 		(pts
+			(xy 215.9 128.27) (xy 215.9 130.81)
+		)
+		(stroke
+			(width 0)
+			(type default)
+		)
+	)
+	(wire
+		(pts
 			(xy 175.26 204.47) (xy 172.72 204.47)
 		)
@@
 	(wire
 		(pts
+			(xy 215.9 120.65) (xy 215.9 118.11)
+		)
+		(stroke
+			(width 0)
+			(type default)
+		)
+	)
+	(wire
+		(pts
 			(xy 381 234.95) (xy 381 237.49)
 		)
@@
 		)
 	)
+	(label "SR_SCK"
+		(at 215.9 118.11 90)
+		(effects
+			(font
+				(size 1.27 1.27)
+			)
+			(justify left bottom)
+		)
+	)
 	(label "NRST"
 		(at 73.66 127 0)
@@
 		)
 	)
-	(label "SR_DATA"
+	(label "LAMP6"
 		(at 73.66 124.46 0)
 		(effects
@@
 		)
 	)
-	(label "LAMP9"
+	(label "SR_SCK"
 		(at 48.26 121.92 180)
 		(effects
@@
 		)
 	)
+	(label "SR_CLK"
+		(at 215.9 130.81 270)
+		(effects
+			(font
+				(size 1.27 1.27)
+			)
+			(justify right bottom)
+		)
+	)
 	(label "SR_DATA"
 		(at 243.84 114.3 180)
@@
 		)
 	)
-	(label "SR_CLK"
+	(label "LAMP9"
 		(at 73.66 132.08 0)
 		(effects
@@
 		)
 	)
-	(label "LAMP6"
+	(label "SR_DATA"
 		(at 48.26 124.46 180)
 		(effects
@@
 					(unit 1)
 				)
+			)
+		)
+	)
+	(symbol
+		(lib_id "Device:R")
+		(at 215.9 124.46 0)
+		(unit 1)
+		(body_style 1)
+		(exclude_from_sim no)
+		(in_bom yes)
+		(on_board yes)
+		(in_pos_files yes)
+		(dnp no)
+		(property "Reference" "R13"
+			(at 220.98 123.19 0)
+			(show_name no)
+			(do_not_autoplace no)
+			(effects
+				(font
+					(size 1.27 1.27)
+				)
+				(justify left)
+			)
+		)
+		(property "Value" "33"
+			(at 220.98 125.73 0)
+			(show_name no)
+			(do_not_autoplace no)
+			(effects
+				(font
+					(size 1.27 1.27)
+				)
+				(justify left)
+			)
+		)
+		(property "Footprint" "Resistor_SMD:R_0402_1005Metric"
+			(at 215.9 124.46 0)
+			(hide yes)
+			(show_name no)
+			(do_not_autoplace no)
+			(effects
+				(font
+					(size 1.27 1.27)
+				)
+			)
+		)
+		(property "Datasheet" "~"
+			(at 215.9 124.46 0)
+			(hide yes)
+			(show_name no)
+			(do_not_autoplace no)
+			(effects
+				(font
+					(size 1.27 1.27)
+				)
+			)
+		)
+		(property "Description" ""
+			(at 215.9 124.46 0)
+			(hide yes)
+			(show_name no)
+			(do_not_autoplace no)
+			(effects
+				(font
+					(size 1.27 1.27)
+				)
+			)
+		)
+		(pin "1"
+		)
+		(pin "2"
+		)
+		(instances
+			(project "NeonPine"
+				(path "/f460b743-0f84-4eb6-8cd0-caf2149a2015"
+					(reference "R13")
+					(unit 1)
+				)
