File: NeonPine.kicad_sch (KiCad schematic)
At the start: 96 parts, among them J1 USB-C 6P (USB4125-GF-A), J2 SWD pogo pads, Q1 DMN15H310SE, Q11 MMDT5551, Q12 MMDT5551, Q13 MMDT5551, Q14 MMDT5551, Q15 MMDT5551, Q16 MMDT5551, Q17 MMDT5551, Q18 MMDT5551, Q19 MMDT5551, Q2 TEPT4400, Q20 MMDT5551, U1 CH32V003F4P6, U2 74HC595BQ, U3 74HC595BQ

Commit message: cheaper components
Parts:
- C1: value 10u -> 10uF
- C10, C2, C6, C7, C9: value 100n -> 100nF
- C3: value 22u 10V -> 22uF 10V
- C4: value 1u 250V -> 1uF 250V
- C5: value 10n -> 10nF
- C8: value 100p C0G 250V -> 100pF 250V C0G
- D1: value 200V 1A fast SOD-123F (verify P/N) -> 200V 1A fast recovery
- D2: MPN (none) -> SMF100A
- D3: value SMF5.0A (TVS) -> SMF5.0A; MPN (none) -> SMF5.0A
- F1: value PTC 0.5A (MF-NSMF050-2) -> MF-NSMF050-2; MPN (none) -> MF-NSMF050-2
- FB1: value 600R@100MHz -> 600Ω@100MHz
- J1: value USB-C 6P (USB4125-GF-A) -> USB4125-GF-A; MPN (none) -> USB4125-GF-A
- J2, TP2, TP3: now left out of the parts list
- L11: value 330u (SWPA6028S331MT, Isat>=0.4A) -> 330uH; MPN (none) -> SWPA6028S331MT
- LA1, LA10, LA2, LA3, LA4, LA5, LA6, LA7, LA8, LA9: MPN (none) -> NEON-3
- Q1: MPN (none) -> DMN15H310SE
- Q11, Q12, Q13, Q14, Q15, Q16, Q17, Q18, Q19, Q20: LCSC (none) -> C148105; MPN (none) -> MMDT5551(RANGE:100-300)
- Q2: MPN (none) -> TEPT4400
- R1: value 47 -> 47Ω
- R11: value 1k -> 1kΩ
- R12: value 100 (snubber) -> 100Ω
- R13: value 33 -> 33Ω
- R2: value 100k -> 100kΩ
- R21, R22, R23, R24, R25, R26, R27, R28, R29, R30, R31, R32, R33, R34, R35, R36, R37, R38, R39, R40: value 150k 200V -> 150kΩ 200V
- R3, R4: value 5k1 -> 5.1kΩ
- R41, R42, R43, R44, R45, R46, R47, R48, R49, R50, R51, R52, R53, R54, R55, R56, R57, R58, R59, R60, R9: value 22k -> 22kΩ
- R5, R6: value 1M -> 1MΩ
- R7: value 39k -> 39kΩ
- U1: MPN (none) -> CH32V003F4P6
- U2, U3: MPN (none) -> 74HC595BQ,115
