File: NeonPine.kicad_sch (KiCad schematic)
At the start: 71 parts, among them J1 USB-C 6P (USB4125-GF-A), J2 SWD pogo pads, Q1 DMN15H310SE, Q11 MMBTA42, Q12 MMBTA42, Q13 MMBTA42, Q14 MMBTA42, Q15 MMBTA42, Q16 MMBTA42, Q17 MMBTA42, Q18 MMBTA42, Q19 MMBTA42, Q2 TEPT4400, Q20 MMBTA42, U1 CH32V003F4P6

Commit message: incomplete big package ver
Parts:
- removed LA2, LA4: NEON-3, NeonPine:Lamp_Neon_Brightmaster_NEON-3_D4x10_P3.0, symbol Device:Lamp_Neon
- removed Q12: MMBTA42, Package_TO_SOT_SMD:SOT-23, symbol Transistor_BJT:Q_NPN_BEC
- added C10, C9: 100n, Capacitor_SMD:C_0603_1608Metric, symbol Device:C
- added LA5: NEON-3, NeonPine:Lamp_Neon_Brightmaster_NEON-3_D4x10_P3.0, symbol Device:Lamp_Neon
- added Q13, Q21, Q26, Q27, Q28, Q29, Q30: MMBTA42, Package_TO_SOT_SMD:SOT-23, symbol Transistor_BJT:Q_NPN_BEC
- added R23, R25, R27, R34, R35, R36, R37, R38, R39, R40: 150k, Resistor_SMD:R_0805_2012Metric, symbol Device:R
- added R42, R43, R44, R46, R48, R51, R52, R53, R54, R55, R56, R57, R58, R59, R60: 22k, Resistor_SMD:R_0402_1005Metric, symbol Device:R
- added U2, U3: 74HC595BQ, Package_DFN_QFN:DHVQFN-16-1EP_2.5x3.5mm_P0.5mm_EP1x2mm, symbol 74xx:74HC595
- D1: value ES1D -> 200V 1A fast SOD-123F (verify P/N); footprint Diode_SMD:D_SMA -> Diode_SMD:D_SOD-123F
- D2: value SMAJ100A -> SMF100A; footprint Diode_SMD:D_SMA -> Diode_SMD:D_SOD-123F
- LA1: renamed from Q11; value MMBTA42 -> NEON-3; footprint Package_TO_SOT_SMD:SOT-23 -> NeonPine:Lamp_Neon_Brightmaster_NEON-3_D4x10_P3.0; symbol Transistor_BJT:Q_NPN_BEC -> Device:Lamp_Neon
- LA3: renamed from R25; value 150k -> NEON-3; footprint Resistor_SMD:R_0805_2012Metric -> NeonPine:Lamp_Neon_Brightmaster_NEON-3_D4x10_P3.0; symbol Device:R -> Device:Lamp_Neon
- LA4: renamed from R46; value 22k -> NEON-3; footprint Resistor_SMD:R_0603_1608Metric -> NeonPine:Lamp_Neon_Brightmaster_NEON-3_D4x10_P3.0; symbol Device:R -> Device:Lamp_Neon
- Q11: renamed from R22; value 150k -> MMBTA42; footprint Resistor_SMD:R_0805_2012Metric -> Package_TO_SOT_SMD:SOT-23; symbol Device:R -> Transistor_BJT:Q_NPN_BEC
- Q12: renamed from R43; value 22k -> MMBTA42; footprint Resistor_SMD:R_0603_1608Metric -> Package_TO_SOT_SMD:SOT-23; symbol Device:R -> Transistor_BJT:Q_NPN_BEC
- Q23: renamed from LA5; value NEON-3 -> MMBTA42; footprint NeonPine:Lamp_Neon_Brightmaster_NEON-3_D4x10_P3.0 -> Package_TO_SOT_SMD:SOT-23; symbol Device:Lamp_Neon -> Transistor_BJT:Q_NPN_BEC
- Q24: renamed from R27; value 150k -> MMBTA42; footprint Resistor_SMD:R_0805_2012Metric -> Package_TO_SOT_SMD:SOT-23; symbol Device:R -> Transistor_BJT:Q_NPN_BEC
- Q25: renamed from R48; value 22k -> MMBTA42; footprint Resistor_SMD:R_0603_1608Metric -> Package_TO_SOT_SMD:SOT-23; symbol Device:R -> Transistor_BJT:Q_NPN_BEC
- R22: renamed from R42; value 22k -> 150k; footprint Resistor_SMD:R_0603_1608Metric -> Resistor_SMD:R_0805_2012Metric
- R31: renamed from LA1; value NEON-3 -> 150k; footprint NeonPine:Lamp_Neon_Brightmaster_NEON-3_D4x10_P3.0 -> Resistor_SMD:R_0805_2012Metric; symbol Device:Lamp_Neon -> Device:R
- R33: renamed from R44; value 22k -> 150k; footprint Resistor_SMD:R_0603_1608Metric -> Resistor_SMD:R_0805_2012Metric
- R41, R45, R47, R49, R50: footprint Resistor_SMD:R_0603_1608Metric -> Resistor_SMD:R_0402_1005Metric
- TP3: value BUZZ/spare -> SR_CLK test
- renumbered LA3 to LA2, Q13 to Q22, R23 to R32
Connections:
- net B2 is gone; now on an unnamed net: R22.2
- net +5V: now also C10.1, C9.1, U2.10 (~{SRCLR}), U2.16 (VCC), U3.10 (~{SRCLR}), U3.16 (VCC)
- net GND: now also Q11.2 (E), Q12.2 (E), Q23.2 (E), Q24.2 (E), Q25.2 (E), C10.2, C9.2, Q13.2 (E), Q21.2 (E), Q26.2 (E), Q27.2 (E), Q28.2 (E), Q29.2 (E), Q30.2 (E), U2.13 (~{OE}), U2.8 (GND), U3.13 (~{OE}), U3.8 (GND); no longer LA1.2 (E)
- net HV+: now also R22.1, R31.1, R33.1, R23.1, R25.1, R27.1, R34.1, R35.1, R36.1, R37.1, R38.1, R39.1, R40.1; no longer LA3.1, Q11.1, Q24.1
- net LAMP1: now also U2.3 (QD); no longer U1.14 (PC4)
- net LAMP10: now also U1.17 (PC7); no longer U1.1 (PD4)
- net LAMP2: now also U1.14 (PC4), R42.1; no longer R22.1, U1.12 (PC2)
- net LAMP3: now also U1.15 (PC5), R43.1; no longer Q12.1, U1.16 (PC6)
- net LAMP4: now also R44.1; no longer R33.1
- net LAMP5: now also U1.12 (PC2); no longer U1.13 (PC3)
- net LAMP6: now also U1.16 (PC6), R46.1; no longer LA4.1, U1.17 (PC7)
- net LAMP8: now also R48.1; no longer Q25.1
- net LAMP9: now also U1.13 (PC3); no longer U1.15 (PC5)
- net at LA3.2: now also Q23.3 (C), R23.2; no longer Q23.2
- net at R21.2: now also LA1.2, Q21.3 (C); no longer R31.2
- net at LA6.1, Q16.3 (C): now also R36.2
- net at LA8.2, R28.2: now also Q28.3 (C)
- net at Q23.1 (B): now also R53.2; no longer Q15.3 (C)
- net at LA10.1, Q20.3 (C): now also R40.2
- net at LA10.2, R30.2: now also Q30.3 (C)
- net at Q14.3 (C): now also LA4.1, R34.2
- net at R24.2: now also LA4.2, Q24.3 (C)
- net at LA2.1: now also Q12.3 (C), R32.2; no longer Q22.3 (C)
- net at LA2.2: now also Q22.3 (C); no longer R32.2
- net at LA7.2: now also Q27.3 (C), R27.2; no longer Q24.2
- net SR_DATA: now reaches U1.3 (PD6)
- net SR_DATA: now also U2.14 (SER)
- net at LA9.1, Q19.3 (C): now also R39.2
- net at LA6.2, R26.2: now also Q26.3 (C)
- net at LA8.1, Q18.3 (C): now also R38.2
- net at LA7.1, Q17.3 (C): now also R37.2
- net at LA9.2, R29.2: now also Q29.3 (C)
- net B1: no longer names the net of LA1.1
- net B1: now also Q11.3 (C), R31.2; no longer R41.2
- net B10: no longer names the net of Q20.1 (B), R50.2
- net B3: no longer names the net of Q22.1 (B)
- net B3: now also R52.2; no longer Q12.2
- net B4: no longer names the net of R33.2
- net B4: now also LA3.1, Q13.3 (C); no longer Q14.1 (B)
- net B5: no longer names the net of Q15.1 (B), R45.2
- net B6: no longer names the net of Q16.1 (B)
- net B6: now also R46.2; no longer LA4.2
- net B7: no longer names the net of Q17.1 (B), R47.2
- net B8: no longer names the net of Q18.1 (B)
- net B8: now also R48.2; no longer Q25.2
- net B9: no longer names the net of Q19.1 (B), R49.2
- net BUZZ renamed SR_CLK
- net SR_CLK: now also U2.11 (SRCLK), U3.11 (SRCLK)
- new net: Q12.1 (B), R42.2
- new net: Q21.1 (B), R51.2
- new net: Q26.1 (B), R56.2
- new net: Q13.1 (B), R43.2
- new net: Q29.1 (B), R59.2
- new net: Q14.1 (B), R44.2
- new net: Q27.1 (B), R57.2
- new net: Q24.1 (B), R54.2
- new net: LA5.1, Q15.3 (C), R35.2
- new net: LA5.2, Q25.3 (C), R25.2
- new net: Q25.1 (B), R55.2
- new net: Q28.1 (B), R58.2
- new net: Q11.1 (B), R41.2
- new net: Q30.1 (B), R60.2
- new net LAMPA1: R51.1, U2.2 (QC)
- new net LAMPA10: R60.1, U3.2 (QC)
- new net LAMPA2: R52.1, U2.1 (QB)
- new net LAMPA3: R53.1, U2.5 (QF)
- new net LAMPA4: R54.1, U2.15 (QA)
- new net LAMPA5: R55.1, U2.4 (QE)
- new net LAMPA6: R56.1, U3.7 (QH)
- new net LAMPA7: R57.1, U2.6 (QG)
- new net LAMPA8: R58.1, U2.7 (QH)
- new net LAMPA9: R59.1, U3.3 (QD)
- new net SR_CHAIN: U2.9 (QH'), U3.14 (SER)
- new net SR_LATCH: U1.1 (PD4), U2.12 (RCLK), U3.12 (RCLK)
- no-connect marks 0 -> 6
Other:
- note added: "I_lamp = (V_HV - 60 V)/150k ≈ 0.1–0.3 mA, plus V_HV/150k ≈ 0.7 mA lost in the pulled-low lead's own pull-up. Both off: dark, no current."
- note added: "LAMP DRIVE – 2 × 74HC595: LAMPA1–10 (anode-side switches) + the one cathode switch the MCU has no pin for"
- note added: "NEON LAMPS – Brightmaster NEON-3 (strike ≤90 VDC, ~60 V settled). Each lead: 150k to HV+ and an MMBTA42 to GND. Pull one lead low: that electrode glows."
- note added: "SR_DATA = PD6, SR_CLK = PA1, SR_LATCH = PD4. /OE tied low: outputs are random until the first latch, but the boost is off then (R2)."
- note removed: "NEON LAMPS – Brightmaster NEON-3 (4x10, strike ≤90 VDC, ~60 V settled): I = (V_HV - 60 V)/150k ≈ 0.1–0.3 mA, MMBTA42 low-side switches"
- moved on the sheet: LA1, LA2, Q22, Q23, R21, R22, R32, R33

Commit message: 2Layer routing complete
needs cleanup
Parts:
- C10, C2, C5, C6, C7, C9: footprint Capacitor_SMD:C_0603_1608Metric -> Capacitor_SMD:C_0402_1005Metric
- Q11: renamed from Q21; value MMBTA42 -> MMDT5551; footprint Package_TO_SOT_SMD:SOT-23 -> Package_TO_SOT_SMD:SOT-363_SC-70-6; symbol Transistor_BJT:Q_NPN_BEC -> Transistor_BJT:Q_Dual_NPN_NPN_E1B1C2E2B2C1
- Q11, Q12, Q13, Q14, Q15, Q16, Q17, Q18, Q19, Q20: value MMBTA42 -> MMDT5551; footprint Package_TO_SOT_SMD:SOT-23 -> Package_TO_SOT_SMD:SOT-363_SC-70-6; symbol Transistor_BJT:Q_NPN_BEC -> Transistor_BJT:Q_Dual_NPN_NPN_E1B1C2E2B2C1
- Q12: renamed from Q22; value MMBTA42 -> MMDT5551; footprint Package_TO_SOT_SMD:SOT-23 -> Package_TO_SOT_SMD:SOT-363_SC-70-6; symbol Transistor_BJT:Q_NPN_BEC -> Transistor_BJT:Q_Dual_NPN_NPN_E1B1C2E2B2C1
- Q13: renamed from Q23; value MMBTA42 -> MMDT5551; footprint Package_TO_SOT_SMD:SOT-23 -> Package_TO_SOT_SMD:SOT-363_SC-70-6; symbol Transistor_BJT:Q_NPN_BEC -> Transistor_BJT:Q_Dual_NPN_NPN_E1B1C2E2B2C1
- Q14: renamed from Q24; value MMBTA42 -> MMDT5551; footprint Package_TO_SOT_SMD:SOT-23 -> Package_TO_SOT_SMD:SOT-363_SC-70-6; symbol Transistor_BJT:Q_NPN_BEC -> Transistor_BJT:Q_Dual_NPN_NPN_E1B1C2E2B2C1
- Q15: renamed from Q25; value MMBTA42 -> MMDT5551; footprint Package_TO_SOT_SMD:SOT-23 -> Package_TO_SOT_SMD:SOT-363_SC-70-6; symbol Transistor_BJT:Q_NPN_BEC -> Transistor_BJT:Q_Dual_NPN_NPN_E1B1C2E2B2C1
- Q16: renamed from Q26; value MMBTA42 -> MMDT5551; footprint Package_TO_SOT_SMD:SOT-23 -> Package_TO_SOT_SMD:SOT-363_SC-70-6; symbol Transistor_BJT:Q_NPN_BEC -> Transistor_BJT:Q_Dual_NPN_NPN_E1B1C2E2B2C1
- Q17: renamed from Q27; value MMBTA42 -> MMDT5551; footprint Package_TO_SOT_SMD:SOT-23 -> Package_TO_SOT_SMD:SOT-363_SC-70-6; symbol Transistor_BJT:Q_NPN_BEC -> Transistor_BJT:Q_Dual_NPN_NPN_E1B1C2E2B2C1
- Q18: renamed from Q28; value MMBTA42 -> MMDT5551; footprint Package_TO_SOT_SMD:SOT-23 -> Package_TO_SOT_SMD:SOT-363_SC-70-6; symbol Transistor_BJT:Q_NPN_BEC -> Transistor_BJT:Q_Dual_NPN_NPN_E1B1C2E2B2C1
- Q19: renamed from Q29; value MMBTA42 -> MMDT5551; footprint Package_TO_SOT_SMD:SOT-23 -> Package_TO_SOT_SMD:SOT-363_SC-70-6; symbol Transistor_BJT:Q_NPN_BEC -> Transistor_BJT:Q_Dual_NPN_NPN_E1B1C2E2B2C1
- Q20: renamed from Q30; value MMBTA42 -> MMDT5551; footprint Package_TO_SOT_SMD:SOT-23 -> Package_TO_SOT_SMD:SOT-363_SC-70-6; symbol Transistor_BJT:Q_NPN_BEC -> Transistor_BJT:Q_Dual_NPN_NPN_E1B1C2E2B2C1
- R1, R11, R2, R3, R4, R7, R9: footprint Resistor_SMD:R_0603_1608Metric -> Resistor_SMD:R_0402_1005Metric
- R21, R22, R23, R24, R25, R26, R27, R28, R29, R30, R31, R32, R33, R34, R35, R36, R37, R38, R39, R40: value 150k -> 150k 200V; footprint Resistor_SMD:R_0805_2012Metric -> Resistor_SMD:R_0603_1608Metric
- U2, U3: footprint Package_DFN_QFN:DHVQFN-16-1EP_2.5x3.5mm_P0.5mm_EP1x2mm -> NeonPine:DHVQFN-16-1EP_2.5x3.5mm_P0.5mm_EP1x2mm_EPGND
Connections:
- net GND: now also Q11.1 (E1), Q11.4 (E2), Q12.1 (E1), Q12.4 (E2), Q13.1 (E1), Q13.4 (E2), Q14.1 (E1), Q14.4 (E2), Q15.1 (E1), Q15.4 (E2), Q16.1 (E1), Q16.4 (E2), Q17.1 (E1), Q17.4 (E2), Q18.1 (E1), Q18.4 (E2), Q19.1 (E1), Q19.4 (E2), Q20.1 (E1), Q20.4 (E2); no longer Q11.2 (E), Q11.2 (E), Q12.2 (E), Q12.2 (E), Q13.2 (E), Q13.2 (E), Q14.2 (E), Q14.2 (E), Q15.2 (E), Q15.2 (E), Q16.2 (E), Q16.2 (E), Q17.2 (E), Q17.2 (E), Q18.2 (E), Q18.2 (E), Q19.2 (E), Q19.2 (E), Q20.2 (E), Q20.2 (E)
- net LAMP1: now also U2.5 (QF); no longer U2.3 (QD)
- net LAMP2: now also U1.12 (PC2); no longer U1.14 (PC4)
- net LAMP3: now also U1.14 (PC4); no longer U1.15 (PC5)
- net LAMP5: now also U1.13 (PC3); no longer U1.12 (PC2)
- net LAMP9: now also U1.15 (PC5); no longer U1.13 (PC3)
- net LAMPA1: now also U2.4 (QE); no longer U2.2 (QC)
- net LAMPA10: now also U3.4 (QE); no longer U3.2 (QC)
- net LAMPA2: now also U2.3 (QD); no longer U2.1 (QB)
- net LAMPA3: now also U2.7 (QH); no longer U2.5 (QF)
- net LAMPA4: now also U2.2 (QC); no longer U2.15 (QA)
- net LAMPA5: now also U2.6 (QG); no longer U2.4 (QE)
- net LAMPA7: now also U2.1 (QB); no longer U2.6 (QG)
- net LAMPA8: now also U2.15 (QA); no longer U2.7 (QH)
- net LAMPA9: now also U3.5 (QF); no longer U3.3 (QD)
- net at LA3.1, R33.2: now also Q13.6 (C1); no longer Q13.3 (C)
- net at R42.2: now also Q12.2 (B1); no longer Q12.1 (B)
- net at LA2.1, R32.2: now also Q12.6 (C1); no longer Q12.3 (C)
- net at R46.2: now also Q16.2 (B1); no longer Q16.1 (B)
- net at R53.2: now also Q13.5 (B2); no longer Q13.1 (B)
- net at R51.2: now also Q11.5 (B2); no longer Q11.1 (B)
- net at R56.2: now also Q16.5 (B2); no longer Q16.1 (B)
- net at R47.2: now also Q17.2 (B1); no longer Q17.1 (B)
- net at LA4.1, R34.2: now also Q14.6 (C1); no longer Q14.3 (C)
- net at LA8.1, R38.2: now also Q18.6 (C1); no longer Q18.3 (C)
- net at R43.2: now also Q13.2 (B1); no longer Q13.1 (B)
- net at R59.2: now also Q19.5 (B2); no longer Q19.1 (B)
- net at LA9.1, R39.2: now also Q19.6 (C1); no longer Q19.3 (C)
- net at R44.2: now also Q14.2 (B1); no longer Q14.1 (B)
- net at R57.2: now also Q17.5 (B2); no longer Q17.1 (B)
- net at LA6.1, R36.2: now also Q16.6 (C1); no longer Q16.3 (C)
- net at R52.2: now also Q12.5 (B2); no longer Q12.1 (B)
- net at R54.2: now also Q14.5 (B2); no longer Q14.1 (B)
- net at LA7.1, R37.2: now also Q17.6 (C1); no longer Q17.3 (C)
- net at R49.2: now also Q19.2 (B1); no longer Q19.1 (B)
- net at LA1.1, R31.2: now also Q11.6 (C1); no longer Q11.3 (C)
- net at R48.2: now also Q18.2 (B1); no longer Q18.1 (B)
- net at R45.2: now also Q15.2 (B1); no longer Q15.1 (B)
- net at R50.2: now also Q20.2 (B1); no longer Q20.1 (B)
- net at LA5.1, R35.2: now also Q15.6 (C1); no longer Q15.3 (C)
- net at R55.2: now also Q15.5 (B2); no longer Q15.1 (B)
- net at R58.2: now also Q18.5 (B2); no longer Q18.1 (B)
- net at LA10.1, R40.2: now also Q20.6 (C1); no longer Q20.3 (C)
- net at R41.2: now also Q11.2 (B1); no longer Q11.1 (B)
- net at R60.2: now also Q20.5 (B2); no longer Q20.1 (B)
Other:
- note added: "NEON LAMPS – Brightmaster NEON-3 (strike ≤90 VDC, ~60 V settled). Each lead: 150k (200 V type) to HV+ and one half of an MMDT5551 (160 V) to GND. Pull one lead low: that electrode glows."
- note removed: "NEON LAMPS – Brightmaster NEON-3 (strike ≤90 VDC, ~60 V settled). Each lead: 150k to HV+ and an MMBTA42 to GND. Pull one lead low: that electrode glows."

Commit message: done
Parts:
- removed C1: 10u, Capacitor_SMD:C_0603_1608Metric, symbol Device:C
- removed C2, C6, C7: 100n, Capacitor_SMD:C_0402_1005Metric, symbol Device:C
- removed D1: 200V 1A fast SOD-123F (verify P/N), Diode_SMD:D_SOD-123F, symbol Device:D
- removed J2: SWD pogo pads, NeonPine:Pogo_1x03_P2.54mm, symbol Connector_Generic:Conn_01x03
- removed LA1, LA10, LA2, LA3, LA4, LA5, LA6, LA7, LA8, LA9: NEON-3, NeonPine:Lamp_Neon_Brightmaster_NEON-3_D4x10_P3.0, symbol Device:Lamp_Neon
- removed Q1: DMN15H310SE, Package_TO_SOT_SMD:SOT-223-3_TabPin2, symbol Transistor_FET:Q_NMOS_GDS
- removed TP2: Touch trunk, NeonPine:TouchPad_D4.0mm_Masked, symbol Connector:TestPoint
- added C3: 22u 10V, Capacitor_SMD:C_0805_2012Metric, symbol Device:C
- added C4: 1u 250V, Capacitor_SMD:C_1210_3225Metric, symbol Device:C
- added D4, D5: BZX884-C3V6, Diode_SMD:D_SOD-882, symbol Device:D_Zener
- added Q2: TEPT4400, LED_THT:LED_D3.0mm, symbol Device:Q_Photo_NPN
- added R1: 47, Resistor_SMD:R_0402_1005Metric, symbol Device:R
- added R13, R14: 68, Resistor_SMD:R_0402_1005Metric, symbol Device:R
- added R15: 1k5, Resistor_SMD:R_0402_1005Metric, symbol Device:R
- added R2: 100k, Resistor_SMD:R_0402_1005Metric, symbol Device:R
- added R21: 150k 200V, Resistor_SMD:R_0603_1608Metric, symbol Device:R
- added R41, R42, R43, R44, R45, R46, R47, R48, R49, R50, R9: 22k, Resistor_SMD:R_0402_1005Metric, symbol Device:R
- C1: renamed from C3; value 22u 10V -> 10u; footprint Capacitor_SMD:C_0805_2012Metric -> Capacitor_SMD:C_0603_1608Metric
- C2: renamed from L11; value 330u (SWPA6028S331MT, Isat>=0.4A) -> 100n; footprint NeonPine:L_6.3x6.3_H3 -> Capacitor_SMD:C_0402_1005Metric; symbol Device:L -> Device:C
- C6: renamed from Q2; value TEPT4400 -> 100n; footprint LED_THT:LED_D3.0mm -> Capacitor_SMD:C_0402_1005Metric; symbol Device:Q_Photo_NPN -> Device:C
- D1: renamed from R2; value 100k -> 200V 1A fast SOD-123F (verify P/N); footprint Resistor_SMD:R_0402_1005Metric -> Diode_SMD:D_SOD-123F; symbol Device:R -> Device:D
- J1: value USB-C 6P (USB4125-GF-A) -> USB-C 16P (USB4105-GF-A); footprint Connector_USB:USB_C_Receptacle_GCT_USB4125-xx-x_6P_TopMnt_Horizontal -> Connector_USB:USB_C_Receptacle_GCT_USB4105-xx-A_16P_TopMnt_Horizontal; symbol Connector:USB_C_Receptacle_PowerOnly_6P -> Connector:USB_C_Receptacle_USB2.0_16P
- J2: renamed from R9; value 22k -> SWD pogo pads; footprint Resistor_SMD:R_0402_1005Metric -> NeonPine:Pogo_1x03_P2.54mm; symbol Device:R -> Connector_Generic:Conn_01x03
- L11: renamed from R1; value 47 -> 330u (SWPA6028S331MT, Isat>=0.4A); footprint Resistor_SMD:R_0402_1005Metric -> NeonPine:L_6.3x6.3_H3; symbol Device:R -> Device:L
- LA1: renamed from Q11; value MMDT5551 -> NEON-3; footprint Package_TO_SOT_SMD:SOT-363_SC-70-6 -> NeonPine:Lamp_Neon_Brightmaster_NEON-3_D4x10_P3.0; symbol Transistor_BJT:Q_Dual_NPN_NPN_E1B1C2E2B2C1 -> Device:Lamp_Neon
- LA10: renamed from Q20; value MMDT5551 -> NEON-3; footprint Package_TO_SOT_SMD:SOT-363_SC-70-6 -> NeonPine:Lamp_Neon_Brightmaster_NEON-3_D4x10_P3.0; symbol Transistor_BJT:Q_Dual_NPN_NPN_E1B1C2E2B2C1 -> Device:Lamp_Neon
- LA2: renamed from Q12; value MMDT5551 -> NEON-3; footprint Package_TO_SOT_SMD:SOT-363_SC-70-6 -> NeonPine:Lamp_Neon_Brightmaster_NEON-3_D4x10_P3.0; symbol Transistor_BJT:Q_Dual_NPN_NPN_E1B1C2E2B2C1 -> Device:Lamp_Neon
- LA3: renamed from Q13; value MMDT5551 -> NEON-3; footprint Package_TO_SOT_SMD:SOT-363_SC-70-6 -> NeonPine:Lamp_Neon_Brightmaster_NEON-3_D4x10_P3.0; symbol Transistor_BJT:Q_Dual_NPN_NPN_E1B1C2E2B2C1 -> Device:Lamp_Neon
- LA4: renamed from Q14; value MMDT5551 -> NEON-3; footprint Package_TO_SOT_SMD:SOT-363_SC-70-6 -> NeonPine:Lamp_Neon_Brightmaster_NEON-3_D4x10_P3.0; symbol Transistor_BJT:Q_Dual_NPN_NPN_E1B1C2E2B2C1 -> Device:Lamp_Neon
- LA5: renamed from Q15; value MMDT5551 -> NEON-3; footprint Package_TO_SOT_SMD:SOT-363_SC-70-6 -> NeonPine:Lamp_Neon_Brightmaster_NEON-3_D4x10_P3.0; symbol Transistor_BJT:Q_Dual_NPN_NPN_E1B1C2E2B2C1 -> Device:Lamp_Neon
- LA6: renamed from Q16; value MMDT5551 -> NEON-3; footprint Package_TO_SOT_SMD:SOT-363_SC-70-6 -> NeonPine:Lamp_Neon_Brightmaster_NEON-3_D4x10_P3.0; symbol Transistor_BJT:Q_Dual_NPN_NPN_E1B1C2E2B2C1 -> Device:Lamp_Neon
- LA7: renamed from Q17; value MMDT5551 -> NEON-3; footprint Package_TO_SOT_SMD:SOT-363_SC-70-6 -> NeonPine:Lamp_Neon_Brightmaster_NEON-3_D4x10_P3.0; symbol Transistor_BJT:Q_Dual_NPN_NPN_E1B1C2E2B2C1 -> Device:Lamp_Neon
- LA8: renamed from Q18; value MMDT5551 -> NEON-3; footprint Package_TO_SOT_SMD:SOT-363_SC-70-6 -> NeonPine:Lamp_Neon_Brightmaster_NEON-3_D4x10_P3.0; symbol Transistor_BJT:Q_Dual_NPN_NPN_E1B1C2E2B2C1 -> Device:Lamp_Neon
- LA9: renamed from Q19; value MMDT5551 -> NEON-3; footprint Package_TO_SOT_SMD:SOT-363_SC-70-6 -> NeonPine:Lamp_Neon_Brightmaster_NEON-3_D4x10_P3.0; symbol Transistor_BJT:Q_Dual_NPN_NPN_E1B1C2E2B2C1 -> Device:Lamp_Neon
- Q1: renamed from C4; value 1u 250V -> DMN15H310SE; footprint Capacitor_SMD:C_1210_3225Metric -> Package_TO_SOT_SMD:SOT-223-3_TabPin2; symbol Device:C -> Transistor_FET:Q_NMOS_GDS
- Q11: renamed from R41; value 22k -> MMDT5551; footprint Resistor_SMD:R_0402_1005Metric -> Package_TO_SOT_SMD:SOT-363_SC-70-6; symbol Device:R -> Transistor_BJT:Q_Dual_NPN_NPN_E1B1C2E2B2C1
- Q12: renamed from R42; value 22k -> MMDT5551; footprint Resistor_SMD:R_0402_1005Metric -> Package_TO_SOT_SMD:SOT-363_SC-70-6; symbol Device:R -> Transistor_BJT:Q_Dual_NPN_NPN_E1B1C2E2B2C1
- Q13: renamed from R43; value 22k -> MMDT5551; footprint Resistor_SMD:R_0402_1005Metric -> Package_TO_SOT_SMD:SOT-363_SC-70-6; symbol Device:R -> Transistor_BJT:Q_Dual_NPN_NPN_E1B1C2E2B2C1
- Q14: renamed from R44; value 22k -> MMDT5551; footprint Resistor_SMD:R_0402_1005Metric -> Package_TO_SOT_SMD:SOT-363_SC-70-6; symbol Device:R -> Transistor_BJT:Q_Dual_NPN_NPN_E1B1C2E2B2C1
- Q15: renamed from R45; value 22k -> MMDT5551; footprint Resistor_SMD:R_0402_1005Metric -> Package_TO_SOT_SMD:SOT-363_SC-70-6; symbol Device:R -> Transistor_BJT:Q_Dual_NPN_NPN_E1B1C2E2B2C1
- Q16: renamed from R46; value 22k -> MMDT5551; footprint Resistor_SMD:R_0402_1005Metric -> Package_TO_SOT_SMD:SOT-363_SC-70-6; symbol Device:R -> Transistor_BJT:Q_Dual_NPN_NPN_E1B1C2E2B2C1
- Q17: renamed from R47; value 22k -> MMDT5551; footprint Resistor_SMD:R_0402_1005Metric -> Package_TO_SOT_SMD:SOT-363_SC-70-6; symbol Device:R -> Transistor_BJT:Q_Dual_NPN_NPN_E1B1C2E2B2C1
- Q18: renamed from R48; value 22k -> MMDT5551; footprint Resistor_SMD:R_0402_1005Metric -> Package_TO_SOT_SMD:SOT-363_SC-70-6; symbol Device:R -> Transistor_BJT:Q_Dual_NPN_NPN_E1B1C2E2B2C1
- Q19: renamed from R49; value 22k -> MMDT5551; footprint Resistor_SMD:R_0402_1005Metric -> Package_TO_SOT_SMD:SOT-363_SC-70-6; symbol Device:R -> Transistor_BJT:Q_Dual_NPN_NPN_E1B1C2E2B2C1
- Q20: renamed from R50; value 22k -> MMDT5551; footprint Resistor_SMD:R_0402_1005Metric -> Package_TO_SOT_SMD:SOT-363_SC-70-6; symbol Device:R -> Transistor_BJT:Q_Dual_NPN_NPN_E1B1C2E2B2C1
- TP2: renamed from R21; value 150k 200V -> Touch trunk; footprint Resistor_SMD:R_0603_1608Metric -> NeonPine:TouchPad_D4.0mm_Masked; symbol Device:R -> Connector:TestPoint
Connections:
- net NRST is gone; now on net SR_DATA: U1.4 (PD7)
- net +5V: now also J2.1 (Pin_1), L11.1, C3.1, Q2.1 (C)
- net GATE: now also Q1.1 (G), R1.2, R2.1; no longer D1.1, L11.2
- net GATE_DRV: now also U1.3 (PD6), R1.1; no longer L11.1, U1.19 (PD2)
- net GND: now also C2.2, C6.2, J1.A1 (GND), J1.B1 (GND), J2.3 (Pin_3), Q1.3 (S), Q11.1 (E1), Q12.1 (E1), Q13.1 (E1), Q14.1 (E1), Q15.1 (E1), Q16.1 (E1), Q17.1 (E1), Q18.1 (E1), Q19.1 (E1), Q20.1 (E1), C3.2, C4.2, D4.2 (A), D5.2 (A), R2.2, R9.2; no longer D1.2, J2.2, LA1.1 (E1), LA10.1 (E1), LA2.1 (E1), LA3.1 (E1), LA4.1 (E1), LA5.1 (E1), LA6.1 (E1), LA7.1 (E1), LA8.1 (E1), LA9.1 (E1), Q1.2
- net HV+: now also D1.1 (K), C4.1, R21.1; no longer Q1.1, TP2.1
- net LAMP1: now also R41.1; no longer Q11.1
- net LAMP10: now also U3.4 (QE), R50.1; no longer Q20.1, U1.17 (PC7)
- net LAMP2: now also R42.1; no longer Q12.1
- net LAMP3: now also R43.1; no longer Q13.1
- net LAMP4: now also R44.1; no longer Q14.1
- net LAMP5: now also R45.1; no longer Q15.1
- net LAMP6: now also R46.1; no longer Q16.1
- net LAMP7: now also R47.1; no longer Q17.1
- net LAMP8: now also R48.1; no longer Q18.1
- net LAMP9: now also R49.1; no longer Q19.1
- net LAMPA10: now also U3.3 (QD); no longer U3.4 (QE)
- net LDR: now also U1.5 (PA1), Q2.2 (E), R9.1; no longer C6.2 (E), J2.1, U1.2 (PD5)
- net SR_CLK: now also U1.17 (PC7); no longer U1.5 (PA1)
- net SR_DATA: no longer U1.3 (PD6)
- net SR_LATCH: now also U1.2 (PD5); no longer U1.1 (PD4)
- net SW: now also D1.2 (A), L11.2, Q1.2 (D); no longer C2.2
- net SWIO: now also J2.2 (Pin_2)
- net VBUS: now also J1.A4 (VBUS), J1.B4 (VBUS), R15.1
- net at R33.2: now also LA3.1, Q13.6 (C1); no longer LA3.6 (C1)
- net at Q13.3 (C2), R23.2: now also LA3.2
- net at Q11.3 (C2): now also LA1.2, R21.2; no longer TP2.2
- net at LA2.2: now also Q12.3 (C2), R22.2; no longer Q12.2
- net at R32.2: now also LA2.1, Q12.6 (C1); no longer LA2.6 (C1)
- net at LA6.2: now also Q16.3 (C2), R26.2; no longer Q16.2
- net at LA7.2: now also Q17.3 (C2), R27.2; no longer Q17.2
- net at Q19.3 (C2), R29.2: now also LA9.2
- net at R34.2: now also LA4.1, Q14.6 (C1); no longer LA4.6 (C1)
- net at Q14.3 (C2), R24.2: now also LA4.2
- net at R38.2: now also LA8.1, Q18.6 (C1); no longer LA8.6 (C1)
- net at Q18.3 (C2), R28.2: now also LA8.2
- net at Q13.2 (B1): now also R43.2; no longer LA3.2 (B1)
- net at R39.2: now also LA9.1, Q19.6 (C1); no longer LA9.6 (C1)
- net at Q14.2 (B1): now also R44.2; no longer LA4.2 (B1)
- net at R36.2: now also LA6.1, Q16.6 (C1); no longer LA6.6 (C1)
- net at Q20.3 (C2), R30.2: now also LA10.2
- net at R37.2: now also LA7.1, Q17.6 (C1); no longer LA7.6 (C1)
- net at Q19.2 (B1): now also R49.2; no longer LA9.2 (B1)
- net at R31.2: now also LA1.1, Q11.6 (C1); no longer LA1.6 (C1)
- net at Q18.2 (B1): now also R48.2; no longer LA8.2 (B1)
- net at LA5.2: now also Q15.3 (C2), R25.2; no longer Q15.2
- net at Q20.2 (B1): now also R50.2; no longer LA10.2 (B1)
- net at R35.2: now also LA5.1, Q15.6 (C1); no longer LA5.6 (C1)
- net at R11.1: now also TP2.1
- net at R40.2: now also LA10.1, Q20.6 (C1); no longer LA10.6 (C1)
- net at Q11.2 (B1): now also R41.2; no longer LA1.2 (B1)
- new net: Q16.2 (B1), R46.2
- new net: Q17.2 (B1), R47.2
- new net: Q12.2 (B1), R42.2
- new net: Q15.2 (B1), R45.2
- new net USB_DM: D5.1 (K), J1.A7 (D-), J1.B7 (D-), R14.2, R15.2
- new net USB_DM_MCU: R14.1, U1.1 (PD4)
- new net USB_DP: D4.1 (K), J1.A6 (D+), J1.B6 (D+), R13.2
- new net USB_DP_MCU: R13.1, U1.19 (PD2)
- no-connect marks 6 -> 7
Other:
- note added: "HV BOOST 75–100 V (MCU-controlled, TIM2_CH3 on PD6, 30 kHz)"
- note added: "LAMP DRIVE – 2 × 74HC595: LAMPA1–10 (anode-side switches) + the cathode switches of LA1 and LA10"
- note added: "PD7 = SR_DATA: program NRST as GPIO (minichlink -D)"
- note added: "SR_DATA = PD7, SR_CLK = PC7, SR_LATCH = PD5. /OE tied low: outputs are random until the first latch, but the boost is off then (R2)."
- note added: "The MCU stays at 5 V: 68R + 3.6 V zeners clamp"
- note added: "USB low-speed (rv003usb): D+ = PD2, D- = PD4."
- note added: "its drive to USB levels. 1k5 D- pull-up to VBUS."
- note removed: "HV BOOST 75–100 V (MCU-controlled, TIM1 30 kHz)"
- note removed: "LAMP DRIVE – 2 × 74HC595: LAMPA1–10 (anode-side switches) + the one cathode switch the MCU has no pin for"
- note removed: "SR_DATA = PD6, SR_CLK = PA1, SR_LATCH = PD4. /OE tied low: outputs are random until the first latch, but the boost is off then (R2)."
- moved on the sheet: C1, LA1, LA10, LA2, LA3, LA4, LA5, LA6, LA7, LA8, LA9
