File: NeonPine-cover.kicad_pcb (KiCad board)
At the start: 2 copper layers, 54.7 x 113.4 mm, 3 parts

Commit message: incomplete big package ver
Other:
- board size 54.7 x 113.4 mm -> 54.7 x 111.4 mm

Commit message: USB clearance fix
Other:
- outline, holes or cut-outs redrawn
Changed lines of the file:
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@@
 	(footprint ""
 		(layer "F.Cu")
-		(at 113 80.5)
+		(at 114.6 107.6)
 		(property "Reference" "H"
 			(at 0 0 0)
@@
 	(footprint ""
 		(layer "F.Cu")
-		(at 87 80.5)
+		(at 113 80.5)
 		(property "Reference" "H"
 			(at 0 0 0)
@@
 	(footprint ""
 		(layer "F.Cu")
-		(at 114.6 107.6)
+		(at 87 80.5)
 		(property "Reference" "H"
 			(at 0 0 0)
@@
 	(gr_line
 		(start 74.143075 96)
-		(end 77.5 96)
+		(end 78.5 96)
 		(stroke
 			(width 0.1)
@@
 	)
 	(gr_line
-		(start 77.5 96)
-		(end 77.833781 96.037608)
-		(stroke
-			(width 0.1)
-			(type default)
-		)
-		(layer "Edge.Cuts")
-	)
-	(gr_line
-		(start 77.833781 96.037608)
-		(end 78.150826 96.148547)
-		(stroke
-			(width 0.1)
-			(type default)
-		)
-		(layer "Edge.Cuts")
-	)
-	(gr_line
-		(start 78.150826 96.148547)
-		(end 78.435235 96.327253)
-		(stroke
-			(width 0.1)
-			(type default)
-		)
-		(layer "Edge.Cuts")
-	)
-	(gr_line
-		(start 78.435235 96.327253)
-		(end 78.672747 96.564765)
-		(stroke
-			(width 0.1)
-			(type default)
-		)
-		(layer "Edge.Cuts")
-	)
-	(gr_line
-		(start 78.672747 96.564765)
-		(end 78.851453 96.849174)
-		(stroke
-			(width 0.1)
-			(type default)
-		)
-		(layer "Edge.Cuts")
-	)
-	(gr_line
-		(start 78.851453 96.849174)
-		(end 78.962392 97.166219)
-		(stroke
-			(width 0.1)
-			(type default)
-		)
-		(layer "Edge.Cuts")
-	)
-	(gr_line
-		(start 78.962392 97.166219)
-		(end 79 97.5)
-		(stroke
-			(width 0.1)
-			(type default)
-		)
-		(layer "Edge.Cuts")
-	)
-	(gr_line
-		(start 79 97.5)
-		(end 79 98)
-		(stroke
-			(width 0.1)
-			(type default)
-		)
-		(layer "Edge.Cuts")
-	)
-	(gr_line
-		(start 79 98)
-		(end 79.037608 98.333781)
-		(stroke
-			(width 0.1)
-			(type default)
-		)
-		(layer "Edge.Cuts")
-	)
-	(gr_line
-		(start 79.037608 98.333781)
-		(end 79.148547 98.650826)
-		(stroke
-			(width 0.1)
-			(type default)
-		)
-		(layer "Edge.Cuts")
-	)
-	(gr_line
-		(start 79.148547 98.650826)
-		(end 79.327253 98.935235)
-		(stroke
-			(width 0.1)
-			(type default)
-		)
-		(layer "Edge.Cuts")
-	)
-	(gr_line
-		(start 79.327253 98.935235)
-		(end 79.564765 99.172747)
-		(stroke
-			(width 0.1)
-			(type default)
-		)
-		(layer "Edge.Cuts")
-	)
-	(gr_line
-		(start 79.564765 99.172747)
-		(end 79.849174 99.351453)
-		(stroke
-			(width 0.1)
-			(type default)
-		)
-		(layer "Edge.Cuts")
-	)
-	(gr_line
-		(start 79.849174 99.351453)
-		(end 80.166219 99.462392)
-		(stroke
-			(width 0.1)
-			(type default)
-		)
-		(layer "Edge.Cuts")
-	)
-	(gr_line
-		(start 80.166219 99.462392)
-		(end 80.5 99.5)
-		(stroke
-			(width 0.1)
-			(type default)
-		)
-		(layer "Edge.Cuts")
-	)
-	(gr_line
-		(start 80.5 99.5)
-		(end 80.833781 99.537608)
-		(stroke
-			(width 0.1)
-			(type default)
-		)
-		(layer "Edge.Cuts")
-	)
-	(gr_line
-		(start 80.833781 99.537608)
-		(end 81.150826 99.648547)
-		(stroke
-			(width 0.1)
-			(type default)
-		)
-		(layer "Edge.Cuts")
-	)
-	(gr_line
-		(start 81.150826 99.648547)
-		(end 81.435235 99.827253)
+		(start 78.5 96)
+		(end 78.691342 96.03806)
+		(stroke
+			(width 0.1)
+			(type default)
+		)
+		(layer "Edge.Cuts")
+	)
+	(gr_line
+		(start 78.691342 96.03806)
+		(end 78.853553 96.146447)
+		(stroke
+			(width 0.1)
+			(type default)
+		)
+		(layer "Edge.Cuts")
+	)
+	(gr_line
+		(start 78.853553 96.146447)
+		(end 78.96194 96.308658)
+		(stroke
+			(width 0.1)
+			(type default)
+		)
+		(layer "Edge.Cuts")
+	)
+	(gr_line
+		(start 78.96194 96.308658)
+		(end 79 96.5)
+		(stroke
+			(width 0.1)
+			(type default)
+		)
+		(layer "Edge.Cuts")
+	)
+	(gr_line
+		(start 79 96.5)
+		(end 79.03806 96.691342)
+		(stroke
+			(width 0.1)
+			(type default)
+		)
+		(layer "Edge.Cuts")
+	)
+	(gr_line
+		(start 79.03806 96.691342)
+		(end 79.146447 96.853553)
+		(stroke
+			(width 0.1)
+			(type default)
+		)
+		(layer "Edge.Cuts")
+	)
+	(gr_line
+		(start 79.146447 96.853553)
+		(end 79.308658 96.96194)
+		(stroke
+			(width 0.1)
+			(type default)
+		)
+		(layer "Edge.Cuts")
+	)
+	(gr_line
+		(start 79.308658 96.96194)
+		(end 79.5 97)
+		(stroke
+			(width 0.1)
+			(type default)
+		)
+		(layer "Edge.Cuts")
+	)
+	(gr_line
+		(start 79.5 97)
+		(end 79.8 97)
+		(stroke
+			(width 0.1)
+			(type default)
+		)
+		(layer "Edge.Cuts")
+	)
+	(gr_line
+		(start 79.8 97)
+		(end 80.047214 97.039155)
+		(stroke
+			(width 0.1)
+			(type default)
+		)
+		(layer "Edge.Cuts")
+	)
+	(gr_line
+		(start 80.047214 97.039155)
+		(end 80.270228 97.152786)
+		(stroke
+			(width 0.1)
+			(type default)
+		)
+		(layer "Edge.Cuts")
+	)
+	(gr_line
+		(start 80.270228 97.152786)
+		(end 80.447214 97.329772)
+		(stroke
+			(width 0.1)
+			(type default)
+		)
+		(layer "Edge.Cuts")
+	)
+	(gr_line
+		(start 80.447214 97.329772)
+		(end 80.560845 97.552786)
+		(stroke
+			(width 0.1)
+			(type default)
+		)
+		(layer "Edge.Cuts")
+	)
+	(gr_line
+		(start 80.560845 97.552786)
+		(end 80.6 97.8)
+		(stroke
+			(width 0.1)
+			(type default)
+		)
+		(layer "Edge.Cuts")
+	)
+	(gr_line
+		(start 80.6 97.8)
+		(end 80.6 98.8)
+		(stroke
+			(width 0.1)
+			(type default)
+		)
+		(layer "Edge.Cuts")
+	)
+	(gr_line
+		(start 80.6 98.8)
+		(end 80.63426 99.016312)
+		(stroke
+			(width 0.1)
+			(type default)
+		)
+		(layer "Edge.Cuts")
+	)
+	(gr_line
+		(start 80.63426 99.016312)
+		(end 80.733688 99.21145)
+		(stroke
+			(width 0.1)
+			(type default)
+		)
+		(layer "Edge.Cuts")
+	)
+	(gr_line
+		(start 80.733688 99.21145)
+		(end 80.88855 99.366312)
+		(stroke
+			(width 0.1)
+			(type default)
+		)
+		(layer "Edge.Cuts")
+	)
+	(gr_line
+		(start 80.88855 99.366312)
+		(end 81.083688 99.46574)
+		(stroke
+			(width 0.1)
+			(type default)
+		)
+		(layer "Edge.Cuts")
+	)
+	(gr_line
+		(start 81.083688 99.46574)
+		(end 81.3 99.5)
 		(stroke
 			(width 0.1)
@@
 	)
 	(gr_line
+		(start 81.3 99.5)
+		(end 81.516312 99.53426)
+		(stroke
+			(width 0.1)
+			(type default)
+		)
+		(layer "Edge.Cuts")
+	)
+	(gr_line
 		(start 81.309982 83.420503)
 		(end 81.458831 83.657511)
@@
 	)
 	(gr_line
-		(start 81.435235 99.827253)
-		(end 81.672747 100.064765)
-		(stroke
-			(width 0.1)
-			(type default)
-		)
-		(layer "Edge.Cuts")
-	)
-	(gr_line
 		(start 81.458831 83.657511)
 		(end 81.668975 83.842358)
@@
 	)
 	(gr_line
+		(start 81.516312 99.53426)
+		(end 81.71145 99.633688)
+		(stroke
+			(width 0.1)
+			(type default)
+		)
+		(layer "Edge.Cuts")
+	)
+	(gr_line
 		(start 81.668975 83.842358)
 		(end 81.923035 83.959758)
@@
 	)
 	(gr_line
-		(start 81.672747 100.064765)
-		(end 81.851453 100.349174)
-		(stroke
-			(width 0.1)
-			(type default)
-		)
-		(layer "Edge.Cuts")
-	)
-	(gr_line
-		(start 81.851453 100.349174)
-		(end 81.962392 100.666219)
+		(start 81.71145 99.633688)
+		(end 81.866312 99.78855)
+		(stroke
+			(width 0.1)
+			(type default)
+		)
+		(layer "Edge.Cuts")
+	)
+	(gr_line
+		(start 81.866312 99.78855)
+		(end 81.96574 99.983688)
 		(stroke
 			(width 0.1)
@@
 	)
 	(gr_line
-		(start 81.962392 100.666219)
-		(end 82 101)
-		(stroke
-			(width 0.1)
-			(type default)
-		)
-		(layer "Edge.Cuts")
-	)
-	(gr_line
-		(start 82 101)
+		(start 81.96574 99.983688)
+		(end 82 100.2)
+		(stroke
+			(width 0.1)
+			(type default)
+		)
+		(layer "Edge.Cuts")
+	)
+	(gr_line
+		(start 82 100.2)
 		(end 82 107.87868)
 		(stroke
